Commit message: update

File: neobot_description/urdf/neobot_urdf.xacro (robot description, xacro)
@@ -67,7 +67,7 @@
   </link>
   <joint name="base_joint" type="fixed">
-      <parent link="base_footprint"/>
-      <child link="base_link" />
-      <origin xyz="0 0 00.0565" rpy="0 0 0"/>
+      <parent link="base_link"/>
+      <child link="base_footprint" />
+      <origin xyz="0 0 -0.0565" rpy="0 0 0"/>
   </joint>
   <joint name="caster_joint" type="fixed">

File: neobot_gazebo/urdf/neobot_gazebo.xacro (robot description, xacro)
@@ -132,5 +132,5 @@
       <odometrySource>world</odometrySource>
       <publishOdomTF>true</publishOdomTF>
-      <robotBaseFrame>base_footprint</robotBaseFrame>
+      <robotBaseFrame>base_link</robotBaseFrame>
       <publishWheelTF>false</publishWheelTF>
       <publishWheelJointState>true</publishWheelJointState>
